File: gausskanone/gausskanone.sch (KiCad schematic (older format))
At the start: 16 parts

Commit message: Doku Flyback
Parts:
- added C? (x2): C, symbol Device:C
- added D?: D_Schottky, symbol Device:D_Schottky
- added Q?: Q_NMOS_DGS, symbol Device:Q_NMOS_DGS
- added R?: R, symbol Device:R
Connections:
- net labels added: +12V, GND
- wire segments 56 -> 74
Other:
- note added: "RC Snubber\n"
Changed lines of the file:
@@
 EESchema Schematic File Version 4
+LIBS:gausskanone-cache
 EELAYER 26 0
 EELAYER END
@@
 	2750 3950 3200 3950
 Wire Wire Line
-	1900 2900 1900 3950
-Wire Wire Line
 	5100 2850 5600 2850
 Wire Wire Line
@@
 	6800 2950 6800 3400
 Connection ~ 6800 3400
+$Comp
+L Device:Q_NMOS_DGS Q?
+U 1 1 5DDDD0BC
+P 2000 5700
+F 0 "Q?" H 2206 5654 50  0000 L CNN
+F 1 "Q_NMOS_DGS" H 2206 5745 50  0000 L CNN
+F 2 "" H 2200 5800 50  0001 C CNN
+F 3 "~" H 2000 5700 50  0001 C CNN
+	1    2000 5700
+	-1   0    0    1
+$EndComp
+$Comp
+L Device:C C?
+U 1 1 5DDDD27D
+P 1250 5450
+F 0 "C?" H 1365 5496 50  0000 L CNN
+F 1 "C" H 1365 5405 50  0000 L CNN
+F 2 "" H 1288 5300 50  0001 C CNN
+F 3 "~" H 1250 5450 50  0001 C CNN
+	1    1250 5450
+	1    0    0    -1
+$EndComp
+$Comp
+L Device:R R?
+U 1 1 5DDDD36E
+P 1500 5200
+F 0 "R?" V 1293 5200 50  0000 C CNN
+F 1 "R" V 1384 5200 50  0000 C CNN
+F 2 "" V 1430 5200 50  0001 C CNN
+F 3 "~" H 1500 5200 50  0001 C CNN
+	1    1500 5200
+	0    1    1    0
+$EndComp
+Wire Wire Line
+	2050 4150 1900 4150
+$Comp
+L power:+12V #PWR?
+U 1 1 5DDDF4C2
+P 3400 4400
+F 0 "#PWR?" H 3400 4250 50  0001 C CNN
+F 1 "+12V" H 3415 4573 50  0000 C CNN
+F 2 "" H 3400 4400 50  0001 C CNN
+F 3 "" H 3400 4400 50  0001 C CNN
+	1    3400 4400
+	1    0    0    -1
+$EndComp
+Wire Wire Line
+	3400 4550 3400 4500
+$Comp
+L Device:C C?
+U 1 1 5DDE0572
+P 3400 4700
+F 0 "C?" H 3515 4746 50  0000 L CNN
+F 1 "C" H 3515 4655 50  0000 L CNN
+F 2 "" H 3438 4550 50  0001 C CNN
+F 3 "~" H 3400 4700 50  0001 C CNN
+	1    3400 4700
+	1    0    0    -1
+$EndComp
+$Comp
+L power:GND #PWR?
+U 1 1 5DDE0649
+P 1900 6250
+F 0 "#PWR?" H 1900 6000 50  0001 C CNN
+F 1 "GND" H 1905 6077 50  0000 C CNN
+F 2 "" H 1900 6250 50  0001 C CNN
+F 3 "" H 1900 6250 50  0001 C CNN
+	1    1900 6250
+	1    0    0    -1
+$EndComp
+Wire Wire Line
+	1350 5200 1250 5200
+Wire Wire Line
+	1250 5200 1250 5300
+Wire Wire Line
+	1650 5200 1900 5200
+Connection ~ 1900 5200
+Wire Wire Line
+	1900 5200 1900 5500
+Wire Wire Line
+	1250 5600 1250 6050
+Wire Wire Line
+	1250 6050 1900 6050
+Wire Wire Line
+	1900 6050 1900 5900
+$Comp
+L Device:D_Schottky D?
+U 1 1 5DDE52A6
+P 1900 3400
+F 0 "D?" V 1854 3479 50  0000 L CNN
+F 1 "D_Schottky" V 1945 3479 50  0000 L CNN
+F 2 "" H 1900 3400 50  0001 C CNN
+F 3 "~" H 1900 3400 50  0001 C CNN
+	1    1900 3400
+	0    1    1    0
+$EndComp
+Wire Wire Line
+	1900 3950 1900 3550
+Wire Wire Line
+	1900 3250 1900 2900
+Wire Wire Line
+	1900 4150 1900 5200
+Wire Wire Line
+	3050 4150 3050 4500
+Wire Wire Line
+	3050 4500 3400 4500
+Wire Wire Line
+	2450 4150 3050 4150
+Connection ~ 3400 4500
+Wire Wire Line
+	3400 4500 3400 4400
+Wire Wire Line
+	1900 6250 1900 6050
+Connection ~ 1900 6050
+Wire Wire Line
+	1900 6050 3400 6050
+Wire Wire Line
+	3400 4850 3400 6050
+Wire Notes Line
+	1650 4900 1650 5600
+Wire Notes Line
+	1650 5600 1050 5600
+Wire Notes Line
+	1050 5600 1050 4900
+Wire Notes Line
+	1050 4900 1650 4900
+Text Notes 1650 4900 2    50   ~ 0
+RC Snubber\n
 $EndSCHEMATC

Commit message: Add files via upload
Parts:
- added C?: 10uF, symbol Device:CP
- added C? (x3): 100nF, symbol Device:CP
- added C? (x2): 22pF, symbol Device:C
- added D?: 1N4001, Diode_THT:D_DO-41_SOD81_P10.16mm_Horizontal, symbol Diode:1N4001
- added J?: Conn_02x03_Counter_Clockwise, symbol Connector_Generic:Conn_02x03_Counter_Clockwise
- added R?: 10k, symbol Device:R
- added SW?: SW_Push, symbol Switch:SW_Push
- added U1: ATmega328-AU, Package_QFP:TQFP-32_7x7mm_P0.8mm, symbol MCU_Microchip_ATmega:ATmega328-AU
- added U?: LM7805_TO220, Package_TO_SOT_THT:TO-220-3_Vertical, symbol Regulator_Linear:LM7805_TO220
- added Y?: Crystal, symbol Device:Crystal
- C2: renamed from C?; value 22M -> 22MF
- C4: renamed from C?; value CP -> 1μF
- U2: renamed from U?; symbol Driver_FET:ACPL-W343 -> gausskanone-rescue:ACPL-W343-Driver_FET
- gave numbers to parts that had none: 18
Connections:
- wire segments 74 -> 165
Other:
- note added: "12V -> 5V\n"
- note added: "Grundschaltung mit Quartz\n"
- note added: "Stützkondensator\n"

Commit message: Added DCDC Converter
Parts:
- removed C1: C, symbol Device:C
- removed L1: L_Coupled, symbol Device:L_Coupled
- removed R1: R, symbol Device:R
- added C?: 1U, symbol Device:C
- added C? (x7): C, symbol Device:C
- added C?: 100N, symbol Device:C
- added C?: CP, symbol Device:CP
- added D?: D_Schottky, symbol Device:D_Schottky
- added D?: 10V, symbol Device:D_Zener
- added R?: Curr Sense, symbol Device:R
- added R? (x7): R, symbol Device:R
- added T?: Transformer_1P_2S, symbol Device:Transformer_1P_2S
- added U?: TPS4021, symbol gausskanone:TPS4021
- U2: symbol gausskanone-rescue:ACPL-W343-Driver_FET -> gausskanone-rescue:ACPL-W343-Driver_FET-gausskanone-rescue
Connections:
- net labels added: DCDC_EN
- wire segments 165 -> 239
Other:
- note added: "Clamping"
- note added: "Compensation Network"
- note added: "Current Sense\nDivider\n"
- note added: "DCDC Diode"
- note added: "Frequency\nSetting\n"
- note added: "Input Filter"
- note added: "Input RC Filter"
- note added: "Soft Start\n"
- note added: "Voltage Divider"
- note removed: "RC Snubber\n"
- moved on the sheet: C2, C3, C4, C?, D1, D2, D3, JP1, L2, Q1, Q2, Q3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

Commit message: Termin 4.12
Parts:
- removed C3: C, symbol Device:C
- removed C?: 10uF, symbol Device:CP
- removed C? (x3): 100nF, symbol Device:CP
- removed C? (x2): 22pF, symbol Device:C
- removed D?: 1N4001, Diode_THT:D_DO-41_SOD81_P10.16mm_Horizontal, symbol Diode:1N4001
- removed J?: Conn_02x03_Counter_Clockwise, symbol Connector_Generic:Conn_02x03_Counter_Clockwise
- removed R?: 10k, symbol Device:R
- removed SW?: SW_Push, symbol Switch:SW_Push
- removed U1: ATmega328-AU, Package_QFP:TQFP-32_7x7mm_P0.8mm, symbol MCU_Microchip_ATmega:ATmega328-AU
- removed U?: LM7805_TO220, Package_TO_SOT_THT:TO-220-3_Vertical, symbol Regulator_Linear:LM7805_TO220
- removed Y?: Crystal, symbol Device:Crystal
- added A?: Arduino_Nano_v3.x, Module:Arduino_Nano, symbol MCU_Module:Arduino_Nano_v3.x
- added D?: D, symbol Device:D
- added D? (x2): LED, symbol Device:LED
- added J?: Conn_01x02_Male, symbol Connector:Conn_01x02_Male
- added J?: Conn_01x03_Male, symbol Connector:Conn_01x03_Male
- added R? (x2): R, symbol Device:R
- added R?: 200R, symbol Device:R
- added R?: 1K, symbol Device:R
- added SW? (x2): SW_DPST, symbol Switch:SW_DPST
- C2: value 22MF -> 22M
- C4: value 1μF -> 1U
Connections:
- net labels added: +5V, READY, TRIGGER
- wire segments 239 -> 207
Other:
- note added: "Manual Trigger"
- note added: "Not Ready"
- note added: "Ready"
- note added: "System Trigger"
- note removed: "12V -> 5V\n"
- note removed: "Grundschaltung mit Quartz\n"
- note removed: "Stützkondensator\n"
- moved on the sheet: C4, D3, R?, TP2, U2, U3

Commit message: Add files via upload
Parts:
- added C? (x2): C, symbol Device:C
- added D?: D_Photo, symbol Device:D_Photo
- added D? (x2): D, symbol Device:D
- added R? (x5): R, symbol Device:R
- added U?: IL300, symbol Isolator_Analog:IL300
- added U? (x3): OP249, symbol Amplifier_Operational:OP249
- U3: value IE1224S -> IE1212S
- U?: symbol gausskanone:TPS4021 -> gausskanone-rescue:TPS4021-gausskanone
Connections:
- wire segments 207 -> 271
Other:
- note added: "An Arduino\n"
- note added: "strombegrenzer\n\n"

Commit message: Termin 11.12
Parts:
- removed D?: D_Photo, symbol Device:D_Photo
- removed J?: Conn_01x02_Male, symbol Connector:Conn_01x02_Male
- removed T?: Transformer_1P_2S, symbol Device:Transformer_1P_2S
- removed U2: U, symbol gausskanone-rescue:ACPL-W343-Driver_FET-gausskanone-rescue
- removed U?: OP249, symbol Amplifier_Operational:OP249
- added C15: CP, symbol Device:CP
- added C16: C, symbol Device:C
- added J2: UC Meas Sec, symbol Connector:Conn_01x03_Female
- added J3: Power Input, symbol Connector:Conn_01x04_Female
- added J4: UC Meas Pri, symbol Connector:Conn_01x03_Female
- added J5: Speedsensor, symbol Connector:Conn_01x04_Male
- added L1: PA6582-AL, symbol Project:PA6582-AL
- added U2: Si8220, Package_SO:SOIC-8_3.9x4.9mm_P1.27mm, symbol Project:Si8220
- added U?: OP249, symbol Amplifier_Operational:OP249
- J1: renamed from J?; value Conn_01x03_Male -> System Bus
- U3: value IE1212S -> IE1212D; footprint (none) -> Project:IEXXXXD
- U7: renamed from U?; footprint (none) -> Project:S-PDSO-G10
- gave numbers to parts that had none: 42
Connections:
- net labels added: IGNITION, ISO+12V, ISO60V, ISOGND, UCADC
- wire segments 271 -> 308
Other:
- note added: "current limiter"
- note removed: "An Arduino\n"
- note removed: "strombegrenzer\n\n"
- moved on the sheet: A1, C10, C11, C12, C13, C14, C3, C5, C6, C7, C8, C9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

Commit message: Changes i made
Parts:
- removed J1: System Bus, symbol Connector:Conn_01x03_Male
- added J?: System Bus, symbol Connector:Conn_01x02_Female
- added U?: DA04-11SRWA, Display_7Segment:DA04-11SURKWA, symbol Display_Character:DA04-11SRWA
Connections:
- net DCDC_EN: now also A1.11 (D8); no longer A1.6 (D3)
- net GND: now also J?.2 (Pin_2), U?.4 (DIG1_CA), U?.5 (DIG2_CA)
- net READY: now also J?.1 (Pin_1)
- net at A1.10 (D7): now also SW1.1, SW1.3; no longer J5.2 (Pin_2)
- net at J5.3 (Pin_3): now also A1.6 (D3); no longer A1.11 (D8)
- net TRIGGER: no longer names the net of A1.8 (D5), SW2.1, SW2.3
- new net: A1.5 (D2), J5.2 (Pin_2)
- now unconnected: U2.3 (CATHODE)
Other:
- moved on the sheet: A1, D10, D11, J5, R15, R20, SW1, SW2

Commit message: Add files via upload
Parts:
- removed C1, C3: C, symbol Device:C
- removed D4, D6: D, symbol Device:D
- removed J2: UC Meas Sec, symbol Connector:Conn_01x03_Female
- removed J4: UC Meas Pri, symbol Connector:Conn_01x03_Female
- removed R1, R10, R5, R7: R, symbol Device:R
- removed U4, U6, U?: OP249, symbol Amplifier_Operational:OP249
- added C?: 100P, symbol Device:C
- added R? (x2): 70K, symbol Device:R
- added R?: 100, symbol Device:R
- added RV?: R_POT, symbol Device:R_POT
- added U?: LT1037, symbol Amplifier_Operational:OP249
- L1: symbol Project:PA6582-AL -> gausskanone-rescue:PA6582-AL-Project
- U2: symbol Project:Si8220 -> gausskanone-rescue:Si8220-Project
Connections:
- net +12V: now also U5.5
- net GND: now also R?.2; no longer U5.5
- net ISO+12V: no longer U5.1
- net ISO60V: now also RV?.3
- net ISOGND: now also U5.2, R?.2
- net at U5.3: now also C?.2, R?.1, U?.2 (-)
- net ISO12V: now reaches U5.4
- net at U5.6: now also R?.1
- net at R6.1: now also RV?.1, U?.3 (+)
- new net: C?.1, R?.2, U?.1
- new net: R?.1, U5.1
Other:
- note added: "VOUT\n"
- note removed: "current limiter"
